Commit message: detection de markers/estimation de pose et calcul des commandes IBVS dans 2 noeuds séparés

File: mobile_platform/platform_description/urdf/mobile_platform.xacro (robot description, xacro)
@@ -35,5 +35,5 @@
             <origin xyz="${origin}"/>
             <axis xyz="${axis}"/>
-            <limit upper="1.57" lower="-1.57" effort="500" velocity="10"/>
+            <limit upper="1.57" lower="-1.57" effort="1000" velocity="10"/>
             <dynamics damping="0.1" friction="0.1"/>
         </joint>
@@ -46,5 +46,5 @@
             <origin xyz="${origin}"/>
             <axis xyz="${axis}"/>
-            <limit upper="3.0" lower="-3.0" effort="500" velocity="10"/>
+            <limit upper="3.0" lower="-3.0" effort="1000" velocity="10"/>
             <dynamics damping="0.1" friction="0.1"/>
         </joint>
